File: PCB_v2/PCB_v2.kicad_sch (KiCad schematic)
At the start: 0 parts

Commit message: pcb-v2
Parts:
- added P1: USB_C_Plug, symbol Connector:USB_C_Plug
- added U1: MIMXRT1062DVJ6B, BGA196_MIMXRT_NXP, symbol MIMXRT1062DVJ6B:MIMXRT1062DVJ6B
- added U3: W25Q32JVZP, Package_SON:WSON-8-1EP_6x5mm_P1.27mm_EP3.4x4.3mm, symbol Memory_Flash:W25Q32JVZP
Connections:
- new net: P1.A1 (GND), P1.A12 (GND), P1.B1 (GND), P1.B12 (GND)
- new net: P1.A4 (VBUS), P1.A9 (VBUS), P1.B4 (VBUS), P1.B9 (VBUS)
- new net VDD_SOC_IN: U1.F6 (VDD_SOC_IN), U1.F7 (VDD_SOC_IN), U1.F8 (VDD_SOC_IN), U1.F9 (VDD_SOC_IN)
Other:
- added sheet accelerometer (accelerometer.kicad_sch)
- added sheet power management (power_management.kicad_sch)
